File: PCB/FriendshipBracelet.kicad_pcb (KiCad board)
At the start: 2 copper layers, 63 x 53.5 mm, 25 parts, among them SW1 SW_Push, U1 XIAO-ESP32-C3-SMD, U2 HS96L03W2C03, U3 ICS-43434_C5656610, U4 ISM303DACTR, U5 SPX3819M5-L-1-8, U6 LSF0108PWR

Commit message: ## July 29th: Mentally fried while desigining case
Parts:
- moved SW1 28.9 mm to (189.0, 69.0)
- moved Vdd1 5.85 mm to (192.5, 73.5)
- moved Vdd_IO1 3.95 mm to (187.5, 73.5)
Routing:
- net Net-(U1-GPIO2_A0_D0): track 31.6 -> 54.5 mm, vias 0 -> 4
- net /1.8V: track 68.4 -> 67.2 mm
